Commit message: Python: dry-run client, working meshes, real tool identity and jog limits
Eight parity gaps from PARITY.md, all in the layer the wire never shows.

## Dry-run client (gap 5)

create_dry_run_client returned None, so Waldo Commander logged "does not
support dry-run simulation" and gave up — no editor path preview, no move
targets, no per-line segments, no timing feasibility, no playback timeline.
The largest single feature loss in the audit.

parol6 runs its real planner in diagnostic mode. par6 has no python binding
to its Rust planner, so rather than invent a second motion model, python/
par6/motion.py ports the runtime's own planning path: ruckig (the reference
implementation of the algorithm par6-motion drives through rsruckig),
TRAPEZOID as a line-by-line port of plan.rs, TOPPRA configured exactly as
the C++ shim configures toppra-cpp, and ports of the cartesian segment and
jog engine with the runtime's own constants. It mirrors the runtime's
refusals too — blend radius, arc/spline/process moves, unhomed planned
motion, non-fitted tools, unreachable poses — so a preview fails where the
arm would.

Correctness is measured against the real thing: the same move_j planned
offline and on a live par6d --sim, at two durations, must agree on window,
landing joints and the shrink between them. A constant or ignored duration
fails it.

## The 3-D viewport was empty (gaps 4, 20)

WC builds package_map from backend_package, but the packaged URDFs said
package://par6_flange/, so every mesh resolved to a path that does not
exist. The sync script now rewrites the package name when it copies, and the
freshness guard compares against that transform rather than raw bytes.

That exposed a second problem: with urdf_path defaulting to the fitted
tool's tree, WC feeds it to pinokin for the workspace envelope and got nq=8
against six joint limits, because the gripper trees declare the jaws as
prismatic arm joints. They are tool DOF — the runtime drives them through
tool_action and reports them as tool status — so the packaged copies demote
them to fixed. The TCP gizmo was also parenting to joint_jaw2.

tools.default came from the config's fitted gripper instead of FLANGE, so
the view has the right tree before the first status frame.

## Tool identity (gaps 8, 10)

robot.tools was keyed upper-case while the wire reports the config spelling,
so robot.tools[status.tool.key] raised KeyError at four WC sites — one of
which then cleared the tool meshes. Canonicalised at the client boundary
only; the wire layer stays a verbatim mirror of par6-proto. A bare
RobotClient now binds the default tools, so rbt.tool.close() in a user
script works.

## Cartesian jog limits were invented (gap 18)

parol6's constants are derived by jacobian-pseudoinverse sampling and pasted
in. par6 now runs the same derivation against its own model and config at
runtime, cached per tool, taking acceleration from the jog ramp's actual
profile rather than parol6's flat 0.8 factor. The test asserts the invariant
rather than the numbers: the angular envelope must tighten at a TCP further
out while the linear one must not.

Tool descriptions come from the gripper TOML's own numbers; joint display
names match parol6's, justified by an identical URDF chain.

Meshes and variants stay empty deliberately, documented at the call site:
the vendor CAD fuses the gripper body into the arm's last link, so a mesh
set would render jaws with no body, and the SSG48 jaw options carry no TCP
or motion data. camera_spec is parity — parol6 defines none either.

python: 149 passed with a live daemon, ruff clean.

Co-Authored-By: Claude Fable 5 <noreply@anthropic.com>
Claude-Session: https://claude.ai/code/session_01GdLL4oE6RejS9yPeSkQXpF

File: python/par6/_data/urdf/par6_flange/urdf/par6_flange.urdf (robot description, URDF)
Before this commit: robot par6_flange, 7 links, 6 joints
Links:
- link base_link: geometry collision mesh filename=package://par6/meshes/base_link.STL; visual mesh filename=package://par6/meshes/base_link.STL
- link elbow: geometry collision mesh filename=package://par6/meshes/elbow.STL; visual mesh filename=package://par6/meshes/elbow.STL
- link gripper: geometry collision mesh filename=package://par6/meshes/gripper.STL; visual mesh filename=package://par6/meshes/gripper.STL
- link lower_arm: geometry collision mesh filename=package://par6/meshes/lower_arm.STL; visual mesh filename=package://par6/meshes/lower_arm.STL
- link shoulder: geometry collision mesh filename=package://par6/meshes/shoulder.STL; visual mesh filename=package://par6/meshes/shoulder.STL
- link upper_arm: geometry collision mesh filename=package://par6/meshes/upper_arm.STL; visual mesh filename=package://par6/meshes/upper_arm.STL
- link wrist: geometry collision mesh filename=package://par6/meshes/wrist.STL; visual mesh filename=package://par6/meshes/wrist.STL

File: python/par6/_data/urdf/par6_msg_gripper/urdf/PAR6_MSG.urdf (robot description, URDF)
Before this commit: robot PAR6_MSG, 10 links, 9 joints
Links:
- link base_link: geometry collision mesh filename=package://par6/meshes/base_link.STL; visual mesh filename=package://par6/meshes/base_link.STL
- link elbow: geometry collision mesh filename=package://par6/meshes/elbow.STL; visual mesh filename=package://par6/meshes/elbow.STL
- link gripper: geometry collision mesh filename=package://par6/meshes/gripper.STL; visual mesh filename=package://par6/meshes/gripper.STL
- link jaw1: geometry collision mesh filename=package://par6/meshes/jaw1.STL; visual mesh filename=package://par6/meshes/jaw1.STL
- link jaw2: geometry collision mesh filename=package://par6/meshes/jaw2.STL; visual mesh filename=package://par6/meshes/jaw2.STL
- link lower_arm: geometry collision mesh filename=package://par6/meshes/lower_arm.STL; visual mesh filename=package://par6/meshes/lower_arm.STL
- link shoulder: geometry collision mesh filename=package://par6/meshes/shoulder.STL; visual mesh filename=package://par6/meshes/shoulder.STL
- link upper_arm: geometry collision mesh filename=package://par6/meshes/upper_arm.STL; visual mesh filename=package://par6/meshes/upper_arm.STL
- link wrist: geometry collision mesh filename=package://par6/meshes/wrist.STL; visual mesh filename=package://par6/meshes/wrist.STL
Joints:
- joint joint_jaw1: type prismatic -> fixed
- joint joint_jaw2: type prismatic -> fixed

File: python/par6/_data/urdf/par6_ssg48_gripper/urdf/par6_ssg48_urdf.urdf (robot description, URDF)
Before this commit: robot par6_ssg48_urdf, 10 links, 9 joints
Links:
- link base_link: geometry collision mesh filename=package://par6/meshes/base_link.STL; visual mesh filename=package://par6/meshes/base_link.STL
- link elbow: geometry collision mesh filename=package://par6/meshes/elbow.STL; visual mesh filename=package://par6/meshes/elbow.STL
- link gripper: geometry collision mesh filename=package://par6/meshes/gripper.STL; visual mesh filename=package://par6/meshes/gripper.STL
- link jaw1: geometry collision mesh filename=package://par6/meshes/jaw1.STL; visual mesh filename=package://par6/meshes/jaw1.STL
- link jaw2: geometry collision mesh filename=package://par6/meshes/jaw2.STL; visual mesh filename=package://par6/meshes/jaw2.STL
- link lower_arm: geometry collision mesh filename=package://par6/meshes/lower_arm.STL; visual mesh filename=package://par6/meshes/lower_arm.STL
- link shoulder: geometry collision mesh filename=package://par6/meshes/shoulder.STL; visual mesh filename=package://par6/meshes/shoulder.STL
- link upper_arm: geometry collision mesh filename=package://par6/meshes/upper_arm.STL; visual mesh filename=package://par6/meshes/upper_arm.STL
- link wrist: geometry collision mesh filename=package://par6/meshes/wrist.STL; visual mesh filename=package://par6/meshes/wrist.STL
Joints:
- joint jaw1_JOINT: type prismatic -> fixed
- joint jaw2_JOINT: type prismatic -> fixed
