Commit message: Close the review's test plan: gaps G3-G13, theatre, lows, and issues #19/#23
The second remediation wave from docs/CODE-REVIEW.md (the first, 9838348,
fixed the criticals/highs/mediums). Eight workstreams, integrated and
verified together:

Homing (G3/G4/G7/G8, L2): a ground-truth reference net — SimBus now
exposes the plant's true joint angle and a multi-boot-pose sweep asserts
the latched home reference against it analytically, the regression net
for the fixed stale-hall and stall-rescale defects. Stall false-positive
guards, the approach timeout, and the release phase's sign, duration and
sample tick are each pinned; the release test re-runs itself with the
config sign inverted to prove it distinguishes sign. PreMove::Idle now
emits real cmd-12 firmware idle plus cmd-28 encoder polls (vendor
Send_Idle semantics) instead of degenerating to the vel-0 keep-alive.

Bus failure (G9, L1): the RT core counts every backend-refused TX/RX
into LoopStats, publishes the backend's LinkHealth, and latches per-node
CanLost => DISABLED when a failure streak spans the freshness window —
driven through a delegating FailingBus over real ticks, with the failure
arm proven allocation-free. The sim dynamics damping constant is
re-derived and CI now builds/tests sim-dynamics.

Gravity (G5/G11): the URDF inertials were a simplified 2.375 kg where
the vendor's own dynamics table says 5.114 kg — transcribed (numbers,
not code) through the numerically-derived frame correspondence, with an
external reference fixture so a simplified URDF fails loudly. Gripper
config inertials now actually feed the gravity model through ToolParams;
changing mass_kg changes the published wrist torque.

Server/protocol (L3/L4/L5, issue #23): link_ok / data_age_ms /
hardware_connected now measure the motor bus (per-node data_age_ticks),
not the server's own snapshot age. A refused fire-and-forget latches as
the standing error while nothing truer stands, so a bad teleport or jog
finally surfaces in error() and STATUS instead of returning success over
an unmoved arm — proven end-to-end, with the jog-burst serialization
guard. Error text: RTI_LINK_LOST's vendor-leftover remedy corrected;
reset-waiter overflow distinguishable from a full motion queue.

CI truth (G2/G6/G10/G12): a vcan job finally EXECUTES the SocketCAN
backend (hard-fail skip semantics under PAR6_REQUIRE_VCAN); a
release-mode soak boots the full runtime at the unpatched 250 Hz shipped
config; jog tests run against a first-order tracking-lag plant and a
live-daemon jog-to-soft-limit e2e; kt-fetch failure shapes covered, plus
an out-of-family plausibility band (a driver answering 10x config is
rejected, not adopted).

Collision enforcement (issue #19): jog/servo streams are now gated — a
StreamGate in the bridge (own coal instance, park resting-pair
exemption) runs parol6's collision_blocked rule with a 0.15 s
velocity-scaled lookahead at datagram admission and re-checks every
housekeeping period while a jog runs; refusals are spoken ERRORs that
ride the new standing-error latch. The escape-depth rule got its
missing half: par6_col_distance in the shim (ABI v5), wired into both
the stream gate and the planner's start-in-collision path. Installation
keep-outs are configurable via [[installation_shapes]] in PAR6.toml
through the same Shape validation path as wire shapes.

Integration surfaced two defects the review missed, both fixed: the sim
driver's velocity-loop integral survived teleport re-seeds and
discharged into the freshly placed plant (the arm landed ~0.03 rad off
every post-jog teleport, ringing); and coal's mesh-pair penetration
depth is nearly flat in true depth, so the escape-depth tolerance is
horizon-scaled for streams and the depth half engages only on
world-shape pairs (full-model distance scans cost ~78 ms — engaging on
marginal arm-arm mesh contacts added 1.6 s to every planned move).
Issue #25 tracks the fidelity follow-ups; issue #24 tracks the
config-theta vs URDF-q coordinate-space finding that must be resolved
before hardware.

Theatre (5.1): the version-constant python test replaced with a real
packaging drift check; the unicast-permanence test now drives a real
send; the ready-pose and gravity-hook tests' claims narrowed to what
they can actually prove.

Verified: fmt, clippy (default + ffi + sim-mujoco + sim-dynamics),
workspace tests both feature states, par6d ffi suite, release 250 Hz
soak, python 148 unit + 16 e2e against the release binary, ruff.

Co-Authored-By: Claude Fable 5 <noreply@anthropic.com>
Claude-Session: https://claude.ai/code/session_01GdLL4oE6RejS9yPeSkQXpF

File: assets/par6_description/URDF/par6_flange/urdf/par6_arm.urdf (robot description, URDF)
Before this commit: robot PAR6_MSG, 10 links, 9 joints
Links:
- removed link jaw1
- removed link jaw2
- removed link tcp
- link base_link: geometry collision mesh filename=package://par6_flange/meshes/base_link.STL; visual mesh filename=package://par6_flange/meshes/base_link.STL
- link elbow: geometry collision mesh filename=package://par6_flange/meshes/elbow.STL; visual mesh filename=package://par6_flange/meshes/elbow.STL
- link gripper: mass 0.167623200457379 -> 0; geometry collision mesh filename=package://par6_flange/meshes/gripper.STL; visual mesh filename=package://par6_flange/meshes/gripper.STL
- link lower_arm: geometry collision mesh filename=package://par6_flange/meshes/lower_arm.STL; visual mesh filename=package://par6_flange/meshes/lower_arm.STL
- link shoulder: geometry collision mesh filename=package://par6_flange/meshes/shoulder.STL; visual mesh filename=package://par6_flange/meshes/shoulder.STL
- link upper_arm: geometry collision mesh filename=package://par6_flange/meshes/upper_arm.STL; visual mesh filename=package://par6_flange/meshes/upper_arm.STL
- link wrist: geometry collision mesh filename=package://par6_flange/meshes/wrist.STL; visual mesh filename=package://par6_flange/meshes/wrist.STL
Joints:
- removed joint joint_jaw1
- removed joint joint_jaw2
- removed joint tcp_fixed_joint
- joint elbow_JOINT: origin xyz=0 -0.18 0 rpy=3.1416 0 -1.5708 -> xyz=0 -0.18 0 rpy=3.14159265358979 0 -1.5707963267949
- joint gripper_JOINT: origin xyz=0 0 0 rpy=1.5708 0 0 -> xyz=0 0 0 rpy=1.5707963267949 0 0
- joint lower_arm_JOINT: origin xyz=0.0435 0 0 rpy=1.5708 0 -3.1416 -> xyz=0.0434999999999984 0 0 rpy=1.5707963267949 0 -3.14159265358979
- joint upper_arm_JOINT: origin xyz=0.023421 0 0.1105 rpy=-1.5708 0 0 -> xyz=0.0234207210610365 0 0.1105 rpy=-1.5707963267949 0 0
- joint wrist_JOINT: origin xyz=0 0 -0.176999999999995 rpy=-1.57079632679489 0 0 -> xyz=0 0 -0.177000000000002 rpy=-1.57079632679489 0 0

File: assets/par6_description/URDF/par6_flange/urdf/par6_flange.urdf (robot description, URDF)
Before this commit: robot par6_flange, 7 links, 6 joints
Links:
- link elbow: mass 0.550970997806044 -> 0.68511
- link gripper: mass 0.024635742513522 -> 0.0555
- link lower_arm: mass 0.382768168076153 -> 0.57956
- link shoulder: mass 0.620900499130961 -> 1.99314
- link upper_arm: mass 0.564255649327409 -> 1.33224
- link wrist: mass 0.230864625594321 -> 0.52381

File: assets/par6_description/URDF/par6_ssg48_gripper/urdf/par6_ssg48_urdf.urdf (robot description, URDF)
Before this commit: robot par6_ssg48_urdf, 10 links, 9 joints
Links:
- link elbow: mass 0.681 -> 0.68511
- link lower_arm: mass 0.579 -> 0.57956
- link shoulder: mass 1.993 -> 1.99314
- link upper_arm: mass 1.332 -> 1.33224
- link wrist: mass 0.523 -> 0.52381

File: python/par6/_data/urdf/par6_flange/urdf/par6_arm.urdf (robot description, URDF)
Before this commit: robot PAR6_MSG, 10 links, 9 joints
Links:
- removed link jaw1
- removed link jaw2
- removed link tcp
- link base_link: geometry collision mesh filename=package://par6/meshes/base_link.STL; visual mesh filename=package://par6/meshes/base_link.STL
- link elbow: geometry collision mesh filename=package://par6/meshes/elbow.STL; visual mesh filename=package://par6/meshes/elbow.STL
- link gripper: mass 0.167623200457379 -> 0; geometry collision mesh filename=package://par6/meshes/gripper.STL; visual mesh filename=package://par6/meshes/gripper.STL
- link lower_arm: geometry collision mesh filename=package://par6/meshes/lower_arm.STL; visual mesh filename=package://par6/meshes/lower_arm.STL
- link shoulder: geometry collision mesh filename=package://par6/meshes/shoulder.STL; visual mesh filename=package://par6/meshes/shoulder.STL
- link upper_arm: geometry collision mesh filename=package://par6/meshes/upper_arm.STL; visual mesh filename=package://par6/meshes/upper_arm.STL
- link wrist: geometry collision mesh filename=package://par6/meshes/wrist.STL; visual mesh filename=package://par6/meshes/wrist.STL
Joints:
- removed joint joint_jaw1
- removed joint joint_jaw2
- removed joint tcp_fixed_joint
- joint elbow_JOINT: origin xyz=0 -0.18 0 rpy=3.1416 0 -1.5708 -> xyz=0 -0.18 0 rpy=3.14159265358979 0 -1.5707963267949
- joint gripper_JOINT: origin xyz=0 0 0 rpy=1.5708 0 0 -> xyz=0 0 0 rpy=1.5707963267949 0 0
- joint lower_arm_JOINT: origin xyz=0.0435 0 0 rpy=1.5708 0 -3.1416 -> xyz=0.0434999999999984 0 0 rpy=1.5707963267949 0 -3.14159265358979
- joint upper_arm_JOINT: origin xyz=0.023421 0 0.1105 rpy=-1.5708 0 0 -> xyz=0.0234207210610365 0 0.1105 rpy=-1.5707963267949 0 0
- joint wrist_JOINT: origin xyz=0 0 -0.176999999999995 rpy=-1.57079632679489 0 0 -> xyz=0 0 -0.177000000000002 rpy=-1.57079632679489 0 0

File: python/par6/_data/urdf/par6_flange/urdf/par6_flange.urdf (robot description, URDF)
Before this commit: robot par6_flange, 7 links, 6 joints
Links:
- link elbow: mass 0.550970997806044 -> 0.68511
- link gripper: mass 0.024635742513522 -> 0.0555
- link lower_arm: mass 0.382768168076153 -> 0.57956
- link shoulder: mass 0.620900499130961 -> 1.99314
- link upper_arm: mass 0.564255649327409 -> 1.33224
- link wrist: mass 0.230864625594321 -> 0.52381

File: python/par6/_data/urdf/par6_msg_gripper/urdf/PAR6_MSG.urdf (robot description, URDF)
Before this commit: robot PAR6_MSG, 10 links, 9 joints
Links:
- link elbow: mass 0.550970997806043 -> 0.68511
- link lower_arm: mass 0.382768168076152 -> 0.57956
- link shoulder: mass 0.620900499130961 -> 1.99314
- link upper_arm: mass 0.564255649327409 -> 1.33224
- link wrist: mass 0.230864625594321 -> 0.52381

File: python/par6/_data/urdf/par6_ssg48_gripper/urdf/par6_ssg48_urdf.urdf (robot description, URDF)
Before this commit: robot par6_ssg48_urdf, 10 links, 9 joints
Links:
- link elbow: mass 0.681 -> 0.68511
- link lower_arm: mass 0.579 -> 0.57956
- link shoulder: mass 1.993 -> 1.99314
- link upper_arm: mass 1.332 -> 1.33224
- link wrist: mass 0.523 -> 0.52381

Commit message: Re-base URDF/MJCF joint coordinates onto the vendor motor convention
Closes the coordinate mismatch of issue #24: every angle in
config/PAR6.toml is vendor theta, but the SolidWorks-exported URDFs
spoke a different joint space (theta = S*q + O, S = [-1,1,-1,-1,1,-1],
O = [0,-pi/2,pi,0,0,0]) and every consumer fed config angles in
verbatim -- self-consistent in sim, wrong against the physical arm
(the configured park pose FK'd 204 mm below the base plane; gravity
feedforward on a torque-controlled machine would have been computed at
a configuration that is not the arm's).

The description tree now speaks theta directly: every revolute axis is
+z and the shoulder/elbow zero offsets are folded into the joint
origins, in all four URDF variants and all four MJCFs (including the
sim scene fork). Link frames, meshes and inertials are untouched;
old-vs-new chains verified frame-for-frame equivalent (<1e-12 URDF,
<1e-7 MJCF at the vendor files' own quat precision) at mapped
configurations, and the park pose now lands at the plausible folded
pose over the base.

Everything recorded or authored against the old coordinates moves with
it:

- golden kinematics + pinokin-sys fixtures regenerated; the gravity
  vendor-reference fixture is remapped exactly (q' = S*q + O,
  tau' = S*tau preserves the vendor-table ground truth; re-verified at
  1e-12 against the re-based model, generator provenance updated).
- collision fixture poses re-authored: three of the old "reachable"
  self-collision poses were outside the arm's real per-joint windows
  (the old generator checked a single symmetric limit); the generator
  now validates against the per-joint soft windows read from
  config/PAR6.toml.
- test postures re-derived where their documented properties no longer
  held on the re-based model: cartesian/curve/sweep starts (IK room
  swept over the soft-limit box), the workspace-edge pose (now blocked
  by the shoulder's soft wall rather than the kinematic singularity,
  where the probe's unclamped DLS blows up), the mujoco grasp pose
  (object re-placed under the same physical jaw approach), the
  torque-plant hold pose (split from CART_START: the extended pose's
  shoulder load exceeds its current authority on feedforward alone).
- the ik-wrap regression posture re-derived so the park-seeded solve
  still turns joints a revolution out of window on this model, and its
  landing tolerance calibrated to the sim's frozen tracking lag (the
  plan lands on the solution exactly; the follow does not).
- config/PAR6.toml, spec/RT.md and the description CHANGELOG now state
  the one-numeric-space convention explicitly.

Full local verification: workspace suite, par6-kin/pinokin-sys ffi
suites, sim-mujoco and sim-dynamics, par6d ffi (13/13), the 250 Hz
release soak, python unit + e2e (16/16), fmt/clippy/ruff.

Co-Authored-By: Claude Fable 5 <noreply@anthropic.com>
Claude-Session: https://claude.ai/code/session_01GdLL4oE6RejS9yPeSkQXpF

File: assets/par6_description/URDF/par6_flange/urdf/par6_arm.urdf (robot description, URDF)
Before this commit: robot par6_arm, 7 links, 6 joints
Joints:
- joint elbow_JOINT: axis 0 0 -1 -> 0 0 1; origin xyz=0 -0.18 0 rpy=3.14159265358979 0 -1.5707963267949 -> xyz=0 -0.18 0 rpy=-3.14159265358979 0 1.57079632679489
- joint gripper_JOINT: axis 0 0 -1 -> 0 0 1
- joint lower_arm_JOINT: axis 0 0 -1 -> 0 0 1
- joint shoulder_JOINT: axis 0 0 -1 -> 0 0 1
- joint upper_arm_JOINT: origin xyz=0.0234207210610365 0 0.1105 rpy=-1.5707963267949 0 0 -> xyz=0.0234207210610365 0 0.1105 rpy=-3.07917384359384 1.57079632679489 -1.50837751679894

File: assets/par6_description/URDF/par6_flange/urdf/par6_flange.urdf (robot description, URDF)
Before this commit: robot par6_flange, 7 links, 6 joints
Joints:
- joint elbow_JOINT: axis 0 0 -1 -> 0 0 1; origin xyz=0 -0.18 0 rpy=3.14159265358979 0 -1.5707963267949 -> xyz=0 -0.18 0 rpy=-3.14159265358979 0 1.57079632679489
- joint gripper_JOINT: axis 0 0 -1 -> 0 0 1
- joint lower_arm_JOINT: axis 0 0 -1 -> 0 0 1
- joint shoulder_JOINT: axis 0 0 -1 -> 0 0 1
- joint upper_arm_JOINT: origin xyz=0.0234207210610365 0 0.1105 rpy=-1.5707963267949 0 0 -> xyz=0.0234207210610365 0 0.1105 rpy=-3.07917384359384 1.57079632679489 -1.50837751679894

File: assets/par6_description/URDF/par6_msg_gripper/urdf/PAR6_MSG.urdf (robot description, URDF)
Before this commit: robot PAR6_MSG, 10 links, 9 joints
Joints:
- joint elbow_JOINT: axis 0 0 -1 -> 0 0 1; origin xyz=0 -0.18 0 rpy=3.1416 0 -1.5708 -> xyz=0 -0.18 0 rpy=3.14158530717959 0 1.57079265358979
- joint gripper_JOINT: axis 0 0 -1 -> 0 0 1
- joint lower_arm_JOINT: axis 0 0 -1 -> 0 0 1
- joint shoulder_JOINT: axis 0 0 -1 -> 0 0 1
- joint upper_arm_JOINT: origin xyz=0.023421 0 0.1105 rpy=-1.5708 0 0 -> xyz=0.023421 0 0.1105 rpy=-3.14159265352934 1.57079265358979 -1.57079632673445

File: assets/par6_description/URDF/par6_ssg48_gripper/urdf/par6_ssg48_urdf.urdf (robot description, URDF)
Before this commit: robot par6_ssg48_urdf, 10 links, 9 joints
Joints:
- joint elbow_JOINT: axis 0 0 -1 -> 0 0 1; origin xyz=0 -0.18 0 rpy=3.1416 0 -1.5708 -> xyz=0 -0.18 0 rpy=3.14158530717959 0 1.57079265358979
- joint gripper_JOINT: axis 0 0 -1 -> 0 0 1
- joint lower_arm_JOINT: axis 0 0 -1 -> 0 0 1
- joint shoulder_JOINT: axis 0 0 -1 -> 0 0 1
- joint upper_arm_JOINT: origin xyz=0.023421 0 0.1105 rpy=-1.5708 0 0 -> xyz=0.023421 0 0.1105 rpy=-3.14159265352934 1.57079265358979 -1.57079632673445

File: python/par6/_data/urdf/par6_flange/urdf/par6_arm.urdf (robot description, URDF)
Before this commit: robot par6_arm, 7 links, 6 joints
Joints:
- joint elbow_JOINT: axis 0 0 -1 -> 0 0 1; origin xyz=0 -0.18 0 rpy=3.14159265358979 0 -1.5707963267949 -> xyz=0 -0.18 0 rpy=-3.14159265358979 0 1.57079632679489
- joint gripper_JOINT: axis 0 0 -1 -> 0 0 1
- joint lower_arm_JOINT: axis 0 0 -1 -> 0 0 1
- joint shoulder_JOINT: axis 0 0 -1 -> 0 0 1
- joint upper_arm_JOINT: origin xyz=0.0234207210610365 0 0.1105 rpy=-1.5707963267949 0 0 -> xyz=0.0234207210610365 0 0.1105 rpy=-3.07917384359384 1.57079632679489 -1.50837751679894

File: python/par6/_data/urdf/par6_flange/urdf/par6_flange.urdf (robot description, URDF)
Before this commit: robot par6_flange, 7 links, 6 joints
Joints:
- joint elbow_JOINT: axis 0 0 -1 -> 0 0 1; origin xyz=0 -0.18 0 rpy=3.14159265358979 0 -1.5707963267949 -> xyz=0 -0.18 0 rpy=-3.14159265358979 0 1.57079632679489
- joint gripper_JOINT: axis 0 0 -1 -> 0 0 1
- joint lower_arm_JOINT: axis 0 0 -1 -> 0 0 1
- joint shoulder_JOINT: axis 0 0 -1 -> 0 0 1
- joint upper_arm_JOINT: origin xyz=0.0234207210610365 0 0.1105 rpy=-1.5707963267949 0 0 -> xyz=0.0234207210610365 0 0.1105 rpy=-3.07917384359384 1.57079632679489 -1.50837751679894

File: python/par6/_data/urdf/par6_msg_gripper/urdf/PAR6_MSG.urdf (robot description, URDF)
Before this commit: robot PAR6_MSG, 10 links, 9 joints
Joints:
- joint elbow_JOINT: axis 0 0 -1 -> 0 0 1; origin xyz=0 -0.18 0 rpy=3.1416 0 -1.5708 -> xyz=0 -0.18 0 rpy=3.14158530717959 0 1.57079265358979
- joint gripper_JOINT: axis 0 0 -1 -> 0 0 1
- joint lower_arm_JOINT: axis 0 0 -1 -> 0 0 1
- joint shoulder_JOINT: axis 0 0 -1 -> 0 0 1
- joint upper_arm_JOINT: origin xyz=0.023421 0 0.1105 rpy=-1.5708 0 0 -> xyz=0.023421 0 0.1105 rpy=-3.14159265352934 1.57079265358979 -1.57079632673445

File: python/par6/_data/urdf/par6_ssg48_gripper/urdf/par6_ssg48_urdf.urdf (robot description, URDF)
Before this commit: robot par6_ssg48_urdf, 10 links, 9 joints
Joints:
- joint elbow_JOINT: axis 0 0 -1 -> 0 0 1; origin xyz=0 -0.18 0 rpy=3.1416 0 -1.5708 -> xyz=0 -0.18 0 rpy=3.14158530717959 0 1.57079265358979
- joint gripper_JOINT: axis 0 0 -1 -> 0 0 1
- joint lower_arm_JOINT: axis 0 0 -1 -> 0 0 1
- joint shoulder_JOINT: axis 0 0 -1 -> 0 0 1
- joint upper_arm_JOINT: origin xyz=0.023421 0 0.1105 rpy=-1.5708 0 0 -> xyz=0.023421 0 0.1105 rpy=-3.14159265352934 1.57079265358979 -1.57079632673445
